File: hardware/scheme/beta2.sch (KiCad schematic (older format))
At the start: 79 parts, among them IC1-1 PIC18F14K50-ESO, IC1-2 PIC18F14K50-ESO, IC2-1 MCP2515-xSO, IC2-2 MCP2515-xSO, IC3-1 MCP2551-I_SN, IC3-2 MCP2551-I_SN, J1 Conn_01x01_Male, J2 Conn_01x01_Male, J3 Conn_01x01_Male, J4 Conn_01x01_Male, J5 Conn_01x01_Male, J6 Conn_01x01_Male, J7 USB_B_Micro, Q1 24Mhz, Q2 24Mhz, Q3 12Mhz, U1 SY6280, U2 GL850G

Commit message: Finished scheme
Scheme finished. Netlist generated. ToDo: place elements in the PCB
Parts:
- removed GND1, GND3: CON3-3, symbol Connector:Conn_01x01_Female
- removed H-1, H-2: CON3-1, symbol Connector:Conn_01x01_Female
- removed L-1, L-2: CON3-2, symbol Connector:Conn_01x01_Female
- added CAN1, CAN2: DB9_Male, Connector_Dsub:DSUB-9_Male_Horizontal_P2.77x2.84mm_EdgePinOffset4.94mm_Housed_MountingHolesOffset7.48mm, symbol Connector:DB9_Male
- added D1: D, Diode_SMD:D_1206_3216Metric_Pad1.42x1.75mm_HandSolder, symbol Device:D
- added R17, R18: 1k, Resistor_SMD:R_1206_3216Metric_Pad1.42x1.75mm_HandSolder, symbol Device:R
- C1, C10, C11, C12, C13, C14, C16, C17, C18, C19, C2, C20, C21, C22, C23, C24, C25, C3, C4, C5, C6, C7, C8, C9, CP1, CP2, CP3, CP4: footprint (none) -> Capacitor_SMD:C_1206_3216Metric_Pad1.42x1.75mm_HandSolder
- C15: value 100nF -> 10uF; footprint (none) -> Capacitor_SMD:C_1206_3216Metric_Pad1.42x1.75mm_HandSolder
- GND1: renamed from J3; footprint (none) -> TestPoint:TestPoint_Pad_D2.5mm
- GND2: renamed from J6; footprint (none) -> TestPoint:TestPoint_Pad_D2.5mm
- H-1: renamed from J1; footprint (none) -> TestPoint:TestPoint_Pad_D2.5mm
- H-2: renamed from J4; footprint (none) -> TestPoint:TestPoint_Pad_D2.5mm
- IC3-1, IC3-2: value MCP2551-I_SN -> MCP2551; footprint SO-8 -> Package_SO:SO-8_5.3x6.2mm_P1.27mm
- J7: footprint (none) -> Connector_USB:USB_Micro-B_Molex-105017-0001
- JP1, JP2, JP3, JP4: footprint (none) -> TestPoint:TestPoint_2Pads_Pitch2.54mm_Drill0.8mm
- L-1: renamed from J2; footprint (none) -> TestPoint:TestPoint_Pad_D2.5mm
- L-2: renamed from J5; footprint (none) -> TestPoint:TestPoint_Pad_D2.5mm
- L1: value 600R/2A -> 600R/200mA; footprint (none) -> Resistor_SMD:R_1206_3216Metric_Pad1.42x1.75mm_HandSolder
- L2, L3, L4, R1, R10, R11, R13, R14, R15, R16, R3, R4, R5, R6, R7, R8, R9: footprint (none) -> Resistor_SMD:R_1206_3216Metric_Pad1.42x1.75mm_HandSolder
- LED1: footprint (none) -> LED_SMD:LED_1206_3216Metric_Pad1.42x1.75mm_HandSolder
- LED2: footprint (none) -> Diode_SMD:D_1206_3216Metric_Pad1.42x1.75mm_HandSolder
- Q1, Q2, Q3: footprint (none) -> Crystal:Crystal_SMD_HC49-SD_HandSoldering
- R12: footprint (none) -> Resistor_SMD:R_0603_1608Metric_Pad1.05x0.95mm_HandSolder
- R2: footprint (none) -> Resistor_SMD:R_2512_6332Metric_Pad1.52x3.35mm_HandSolder
- U1: footprint (none) -> Package_TO_SOT_SMD:SOT-23-5_HandSoldering
- U2: footprint (none) -> Package_SO:SSOP-28_5.3x10.2mm_P0.65mm
Connections:
- net GND: now also CAN1.3, CAN2.3
- net at H-2.1 (Pin_1), IC3-2.7 (CANH): now also R15.2, CAN1.7; no longer JP2.2
- net at IC3-2.6 (CANL), L-2.1 (Pin_1): now also JP2.2, CAN1.2; no longer R15.2
- net at IC1-2.12 (RB5/IOCB5/AN11/RX/DT): now also R18.1; no longer LED2.2 (A)
- net at H-1.1 (Pin_1), IC3-1.7 (CANH): now also R4.2, CAN2.7; no longer JP1.2
- net at IC3-1.6 (CANL), L-1.1 (Pin_1): now also JP1.2, CAN2.2; no longer R4.2
- net at IC1-1.12 (RB5/IOCB5/AN11/RX/DT): now also R17.1; no longer LED1.2 (A)
- net at C7.1, U1.4 (EN), U1.5 (IN): now also D1.1 (K); no longer J7.1 (VBUS), R11.2
- net at U2.1 (AVDD): now also C23.1, C24.1, C25.1, L4.2, U2.10 (AVDD), U2.5 (AVDD)
- new net: LED2.2 (A), R18.2
- new net: LED1.2 (A), R17.2
- new net: D1.2 (A), J7.1 (VBUS), R11.2
- no-connect marks 23 -> 36
Other:
- note added: "Can Interface 1"
- note added: "Can Interface 2"
- moved on the sheet: J7, L1, LED1, LED2
