File: hardware/scheme/cret.sch (KiCad schematic (older format))
At the start: 78 parts, among them IC1-1 PIC18F14K50-ESO, IC1-2 PIC18F14K50-ESO, IC2-1 MCP2515-xSO, IC2-2 MCP2515-xSO, IC3-1 MCP2551, IC3-2 MCP2551, J7 USB_B_Micro, Q1 24Mhz, Q2 24Mhz, Q3 12Mhz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

Commit message: Hardware finished
Scheme reviewed and finished. PCB reviewed and finished. Generated netlist and gerber files. The PCB has been ordered.
Parts:
- LED2: footprint Diode_SMD:D_1206_3216Metric_Pad1.42x1.75mm_HandSolder -> LED_SMD:LED_1206_3216Metric_Pad1.42x1.75mm_HandSolder
- R12: footprint Resistor_SMD:R_0603_1608Metric_Pad1.05x0.95mm_HandSolder -> Resistor_SMD:R_1206_3216Metric_Pad1.42x1.75mm_HandSolder
- R2: footprint Resistor_SMD:R_2512_6332Metric_Pad1.52x3.35mm_HandSolder -> Resistor_SMD:R_1206_3216Metric_Pad1.42x1.75mm_HandSolder
- renumbered CAN2 to CAN1, CAN1 to CAN2
Connections:
- net V1: now also C1.1, C2.1, C3.1, C8.2, CP1.1, IC2-1.18 (VDD), L2.2, R3.1; no longer C9.2, L3.2
- net V2: now also C4.1, C5.1, C6.1, C9.2, CP2.1, IC2-2.18 (VDD), L3.2, R14.1; no longer C8.2, L2.2
- removed net +5V: C1.1, C2.1, C3.1, C4.1, C5.1, C6.1, CP1.1, CP2.1, IC2-1.18 (VDD), IC2-2.18 (VDD), R14.1, R3.1
Other:
- note added: "0.1"
- note added: "19/12/2018"
- note added: "Adrián Marcos"
